File: src/H81-Custom-MotherBoard.kicad_pcb (KiCad board)
At the start: 4 copper layers, 930 parts, among them K1 K1_ICT/X, K2 K1_ICT/X, K3 K1_ICT/X, K4 K1_ICT/X, K5 K1_ICT/X, K6 K1_ICT/X, P2 FAN/1*4/WH/A3/PA66, Q11 MASK/MMBT2222A/SOT23/600mA/40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, Q28 2N7002/SOT23/25pF/5, Q29 MMBT2222A/SOT23/600mA/40, Q30 MMBT2222A/SOT23/600mA/40, Q42 AP431N/SOT23/150mA/X, Q47 2N7002/SOT23/25pF/5, Q48 2N7002/SOT23/25pF/5, Q53 NTMFS4C10NT1G/PPAK/970pF/7.3m, Q57 MASK/MMBT2222A/SOT23/600mA/40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, Q59 MASK/MMBT2222A/SOT23/600mA/40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, Q61 L1085DG/TO252/5A, Q65 BAT54C/SOT23/200mA/X, Q66 MASK/MMBT2222A/SOT23/600mA/40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, Q67 MASK/PMBT2907A/SOT23/-600mA/5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, Q69 P2003ED/P/TO252/30m, Q73 MASK/MMBT2222A/SOT23/600mA/40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, Q83 MASK/MMBT2222A/SOT23/600mA/40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, Q84 MASK/MMBT2222A/SOT23/600mA/40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, Q86 2N7002/SOT23/25pF/5, Q87 MMBT2222A/SOT23/600mA/40, Q9 MMBT2222A/SOT23/600mA/40, U1 LM358DR/SO8, U18 20K/4/1/X, U6 RT9199PSP/SO8/1.8A, U8 SATA2/7/BK/H/OP/VA/D/1/B, U8#2 RT8120DGS/SOP8, Y41 HOLE_3/X

Commit message: .
Parts:
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Connections:
- net +12V renamed /+12V
- net +12V_LOAD renamed /+12V_LOAD
- net -12V renamed /-12V
- net -CASEOPEN renamed /-CASEOPEN
- net -CSA0 renamed /-CSA0
- net -CSA1 renamed /-CSA1
- net -CSB0 renamed /-CSB0
- net -CSB1 renamed /-CSB1
- net -DCLKA0 renamed /-DCLKA0
- net -DCLKA1 renamed /-DCLKA1
- net -DCLKB0 renamed /-DCLKB0
- net -DCLKB1 renamed /-DCLKB1
- net -DDR3_RST renamed /-DDR3_RST
- net -DQSA0 renamed /-DQSA0
- net -DQSA1 renamed /-DQSA1
- net -DQSA2 renamed /-DQSA2
- net -DQSA3 renamed /-DQSA3
- net -DQSA4 renamed /-DQSA4
- net -DQSA5 renamed /-DQSA5
- net -DQSA6 renamed /-DQSA6
- net -DQSA7 renamed /-DQSA7
- net -DQSB0 renamed /-DQSB0
- net -DQSB1 renamed /-DQSB1
- net -DQSB2 renamed /-DQSB2
- net -DQSB3 renamed /-DQSB3
- net -DQSB4 renamed /-DQSB4
- net -DQSB5 renamed /-DQSB5
- net -DQSB6 renamed /-DQSB6
- net -DQSB7 renamed /-DQSB7
- net -D_GPIO_HRST renamed /-D_GPIO_HRST
- net -HOLD0 renamed /-HOLD0
- net -HOLD1 renamed /-HOLD1
- net -PCIE_RST renamed /-PCIE_RST
- net -PCIRSTIN renamed /-PCIRSTIN
- net -PFMRST2 renamed /-PFMRST2
- net -PROCHOT_CON renamed /-PROCHOT_CON
- net -PSON renamed /-PSON
- net -PVIDALRT renamed /-PVIDALRT
- net -PWRBTSW renamed /-PWRBTSW
- net -PWRBT_1 renamed /-PWRBT_1
- net -RST renamed /-RST
- net -RST_BTN renamed /-RST_BTN
- net -SCASA renamed /-SCASA
- net -SCASB renamed /-SCASB
- net -SPI_CS_1 renamed /-SPI_CS_1
- net -SPI_CS_2 renamed /-SPI_CS_2
- net -SPI_HOLD_B renamed /-SPI_HOLD_B
- net -SPI_HOLD_M renamed /-SPI_HOLD_M
- net -SRASA renamed /-SRASA
- net -SRASB renamed /-SRASB
- net -SWEA renamed /-SWEA
- net -SWEB renamed /-SWEB
- net 0_8LEVEL_DDR renamed /0_8LEVEL_DDR
- net 15G renamed /15G
- net 15HG renamed /15HG
- net 1_5LG renamed /1_5LG
- net 28_3VSB renamed /28_3VSB
- net 2_5LEVEL renamed /2_5LEVEL
- net 3VDUAL renamed /3VDUAL
- net 3VDUAL_PCH renamed /3VDUAL_PCH
- net 5VAUX_SW renamed /5VAUX_SW
- net 5VDUAL renamed /5VDUAL
- net 5VSB renamed /5VSB
- net 6609_VCC renamed /6609_VCC
- net 95812_FB renamed /95812_FB
- net 95812_FB_R renamed /95812_FB_R
- net 95812_VDD renamed /95812_VDD
- net 95812_VDDP renamed /95812_VDDP
- net 95812_VIN renamed /95812_VIN
- net AGND renamed /AGND
- net AJ_A2 renamed /AJ_A2
- net AJ_A5 renamed /AJ_A5
- net AJ_B2 renamed /AJ_B2
- net AJ_B5 renamed /AJ_B5
- net AVDD renamed /AVDD
- net A_-CPURST renamed /A_-CPURST
- net A_-HPRDY renamed /A_-HPRDY
- net A_-PROCHOT renamed /A_-PROCHOT
- net A_-SKTOCC renamed /A_-SKTOCC
- net A_-THRMTRIP renamed /A_-THRMTRIP
- net A_-TRST renamed /A_-TRST
- net A_DDR_COMP0 renamed /A_DDR_COMP0
- net A_DDR_COMP1 renamed /A_DDR_COMP1
- net A_DDR_COMP2 renamed /A_DDR_COMP2
- net A_DMI_0RXN renamed /A_DMI_0RXN
- net A_DMI_0RXP renamed /A_DMI_0RXP
- net A_DMI_0TXN renamed /A_DMI_0TXN
- net A_DMI_0TXP renamed /A_DMI_0TXP
- net A_DMI_1RXN renamed /A_DMI_1RXN
- net A_DMI_1RXP renamed /A_DMI_1RXP
- net A_DMI_1TXN renamed /A_DMI_1TXN
- net A_DMI_1TXP renamed /A_DMI_1TXP
- net A_DMI_2RXN renamed /A_DMI_2RXN
- net A_DMI_2RXP renamed /A_DMI_2RXP
- net A_DMI_2TXN renamed /A_DMI_2TXN
- net A_DMI_2TXP renamed /A_DMI_2TXP
- net A_DMI_3RXN renamed /A_DMI_3RXN
- net A_DMI_3RXP renamed /A_DMI_3RXP
- net A_DMI_3TXN renamed /A_DMI_3TXN
- net A_DMI_3TXP renamed /A_DMI_3TXP
- net A_HSW_CFG_RCOMP renamed /A_HSW_CFG_RCOMP
- net A_PECI renamed /A_PECI
- net A_PMSYNC renamed /A_PMSYNC
- net A_PWR_DEBUG renamed /A_PWR_DEBUG
- net A_SM_VREF renamed /A_SM_VREF
- net A_SO renamed /A_SO
- net A_SYC renamed /A_SYC
- net A_TCK renamed /A_TCK
- net A_TESTLOW_1 renamed /A_TESTLOW_1
- net A_TESTLOW_2 renamed /A_TESTLOW_2
- net BEEP- renamed /BEEP-
- net BOOT renamed /BOOT
- net CEB_N renamed /CEB_N
- net CKEA0 renamed /CKEA0
- net CKEA1 renamed /CKEA1
- net CKEB0 renamed /CKEB0
- net CKEB1 renamed /CKEB1
- net CK_-DOTCLK renamed /CK_-DOTCLK
- net CK_-SRCCLK_PCH renamed /CK_-SRCCLK_PCH
- net CK_-SRCCLK_SATA renamed /CK_-SRCCLK_SATA
- net CK_DOTCLK renamed /CK_DOTCLK
- net CK_SRCCLK_PCH renamed /CK_SRCCLK_PCH
- net CK_SRCCLK_SATA renamed /CK_SRCCLK_SATA
- net COUPON1 renamed /COUPON1
- net COUPON2 renamed /COUPON2
- net CPU_VAXG renamed /CPU_VAXG
- net CPU_VTT_OR renamed /CPU_VTT_OR
- net C_-ACZ_RST renamed /C_-ACZ_RST
- net C_ACZ_BITCLK renamed /C_ACZ_BITCLK
- net C_ACZ_SDIN2 renamed /C_ACZ_SDIN2
- net C_ACZ_SDOUT renamed /C_ACZ_SDOUT
- net C_ACZ_SYNC renamed /C_ACZ_SYNC
- net DCLKA0 renamed /DCLKA0
- net DCLKA1 renamed /DCLKA1
- net DCLKB0 renamed /DCLKB0
- net DCLKB1 renamed /DCLKB1
- net DDRVTT renamed /DDRVTT
- net DDR_15V renamed /DDR_15V
- net DDR_15VIO renamed /DDR_15VIO
- net DDR_EN_CON renamed /DDR_EN_CON
- net DDR_VTT_REF renamed /DDR_VTT_REF
- net DMI_COMP renamed /DMI_COMP
- net DQSA0 renamed /DQSA0
- net DQSA1 renamed /DQSA1
- net DQSA2 renamed /DQSA2
- net DQSA3 renamed /DQSA3
- net DQSA4 renamed /DQSA4
- net DQSA5 renamed /DQSA5
- net DQSA6 renamed /DQSA6
- net DQSA7 renamed /DQSA7
- net DQSB0 renamed /DQSB0
- net DQSB1 renamed /DQSB1
- net DQSB2 renamed /DQSB2
- net DQSB3 renamed /DQSB3
- net DQSB4 renamed /DQSB4
- net DQSB5 renamed /DQSB5
- net DQSB6 renamed /DQSB6
- net DQSB7 renamed /DQSB7
- net FAN1_SET renamed /FAN1_SET
- net FAN1_VOUT renamed /FAN1_VOUT
- net FANIO1 renamed /FANIO1
- net FANIO2 renamed /FANIO2
- net FANPWM1 renamed /FANPWM1
- net FANPWM2 renamed /FANPWM2
- net FAUDIO_JD renamed /FAUDIO_JD
- net FDI_CSYNC renamed /FDI_CSYNC
- net FDI_INT renamed /FDI_INT
- net FDI_RCOMP renamed /FDI_RCOMP
- net FDI_TXN0 renamed /FDI_TXN0
- net FDI_TXN1 renamed /FDI_TXN1
- net FDI_TXP0 renamed /FDI_TXP0
- net FDI_TXP1 renamed /FDI_TXP1
- net FRONT_JD renamed /FRONT_JD
- net FUSEVCC_F renamed /FUSEVCC_F
- net FUSEVCC_R renamed /FUSEVCC_R
- net FUSEVCC_USB3_R3 renamed /FUSEVCC_USB3_R3
- net GND renamed /GND
- net GP24 renamed /GP24
- net GP25 renamed /GP25
- net GP26 renamed /GP26
- net GRCOMP renamed /GRCOMP
- net HD+ renamed /HD+
- net H_SYNC renamed /H_SYNC
- net IO_EN1 renamed /IO_EN1
- net ISEN1 renamed /ISEN1
- net ISEN2 renamed /ISEN2
- net ISEN3 renamed /ISEN3
- net ITE_PWROK1 renamed /ITE_PWROK1
- net IT_AVCC renamed /IT_AVCC
- net IT_VCCH renamed /IT_VCCH
- net JP2 renamed /JP2
- net JP3 renamed /JP3
- net JP4 renamed /JP4
- net JP5 renamed /JP5
- net KBCLK renamed /KBCLK
- net KBDATA renamed /KBDATA
- net KCLK renamed /KCLK
- net KDAT renamed /KDAT
- net L2-L renamed /L2-L
- net L2-R renamed /L2-R
- net L2_L renamed /L2_L
- net L2_R renamed /L2_R
- net LAN_3VDUAL_LED renamed /LAN_3VDUAL_LED
- net LA_-SRCCLK_LAN renamed /LA_-SRCCLK_LAN
- net LA_CLKREQB renamed /LA_CLKREQB
- net LA_DVDD10 renamed /LA_DVDD10
- net LA_LED_ACT_TXRX renamed /LA_LED_ACT_TXRX
- net LA_LED_D2 renamed /LA_LED_D2
- net LA_LED_LINK100 renamed /LA_LED_LINK100
- net LA_LED_LINK1000 renamed /LA_LED_LINK1000
- net LA_MDI0+ renamed /LA_MDI0+
- net LA_MDI0- renamed /LA_MDI0-
- net LA_MDI1+ renamed /LA_MDI1+
- net LA_MDI1- renamed /LA_MDI1-
- net LA_MDI2+ renamed /LA_MDI2+
- net LA_MDI2- renamed /LA_MDI2-
- net LA_MDI3+ renamed /LA_MDI3+
- net LA_MDI3- renamed /LA_MDI3-
- net LA_ML_IN renamed /LA_ML_IN
- net LA_ML_IN_C renamed /LA_ML_IN_C
- net LA_ML_IP renamed /LA_ML_IP
- net LA_ML_IP_C renamed /LA_ML_IP_C
- net LA_ML_ON renamed /LA_ML_ON
- net LA_ML_ON_C renamed /LA_ML_ON_C
- net LA_ML_OP renamed /LA_ML_OP
- net LA_ML_OP_C renamed /LA_ML_OP_C
- net LA_REGOUT renamed /LA_REGOUT
- net LA_RSET renamed /LA_RSET
- net LA_SRCCLK_LAN renamed /LA_SRCCLK_LAN
- net LA_VDD33 renamed /LA_VDD33
- net LA_XTALI renamed /LA_XTALI
- net LA_XTALO renamed /LA_XTALO
- net LG1_1 renamed /LG1_1
- net LG2_1 renamed /LG2_1
- net LG3 renamed /LG3
- net LG3_1 renamed /LG3_1
- net LINE1_JD renamed /LINE1_JD
- net LINE2_L renamed /LINE2_L
- net LINE2_R renamed /LINE2_R
- net LINE2_VREFO renamed /LINE2_VREFO
- net LINE_IN_L renamed /LINE_IN_L
- net LINE_IN_R renamed /LINE_IN_R
- net LINE_O_L renamed /LINE_O_L
- net LINE_O_R renamed /LINE_O_R
- net M2_L renamed /M2_L
- net M2_R renamed /M2_R
- net MAAA0 renamed /MAAA0
- net MAAA1 renamed /MAAA1
- net MAAA10 renamed /MAAA10
- net MAAA11 renamed /MAAA11
- net MAAA12 renamed /MAAA12
- net MAAA13 renamed /MAAA13
- net MAAA14 renamed /MAAA14
- net MAAA15 renamed /MAAA15
- net MAAA2 renamed /MAAA2
- net MAAA3 renamed /MAAA3
- net MAAA4 renamed /MAAA4
- net MAAA5 renamed /MAAA5
- net MAAA6 renamed /MAAA6
- net MAAA7 renamed /MAAA7
- net MAAA8 renamed /MAAA8
- net MAAA9 renamed /MAAA9
- net MAAB0 renamed /MAAB0
- net MAAB1 renamed /MAAB1
- net MAAB10 renamed /MAAB10
- net MAAB11 renamed /MAAB11
- net MAAB12 renamed /MAAB12
- net MAAB13 renamed /MAAB13
- net MAAB14 renamed /MAAB14
- net MAAB15 renamed /MAAB15
- net MAAB2 renamed /MAAB2
- net MAAB3 renamed /MAAB3
- net MAAB4 renamed /MAAB4
- net MAAB5 renamed /MAAB5
- net MAAB6 renamed /MAAB6
- net MAAB7 renamed /MAAB7
- net MAAB8 renamed /MAAB8
- net MAAB9 renamed /MAAB9
- net MB_ID2 renamed /MB_ID2
- net MCLK renamed /MCLK
- net MDA0 renamed /MDA0
- net MDA1 renamed /MDA1
- net MDA10 renamed /MDA10
- net MDA11 renamed /MDA11
- net MDA12 renamed /MDA12
- net MDA13 renamed /MDA13
- net MDA14 renamed /MDA14
- net MDA15 renamed /MDA15
- net MDA16 renamed /MDA16
- net MDA17 renamed /MDA17
- net MDA18 renamed /MDA18
- net MDA19 renamed /MDA19
- net MDA2 renamed /MDA2
- net MDA20 renamed /MDA20
- net MDA21 renamed /MDA21
- net MDA22 renamed /MDA22
- net MDA23 renamed /MDA23
- net MDA24 renamed /MDA24
- net MDA25 renamed /MDA25
- net MDA26 renamed /MDA26
- net MDA27 renamed /MDA27
- net MDA28 renamed /MDA28
- net MDA29 renamed /MDA29
- net MDA3 renamed /MDA3
- net MDA30 renamed /MDA30
- net MDA31 renamed /MDA31
- net MDA32 renamed /MDA32
- net MDA33 renamed /MDA33
- net MDA34 renamed /MDA34
- net MDA35 renamed /MDA35
- net MDA36 renamed /MDA36
- net MDA37 renamed /MDA37
- net MDA38 renamed /MDA38
- net MDA39 renamed /MDA39
- net MDA4 renamed /MDA4
- net MDA40 renamed /MDA40
- net MDA41 renamed /MDA41
- net MDA42 renamed /MDA42
- net MDA43 renamed /MDA43
- net MDA44 renamed /MDA44
- net MDA45 renamed /MDA45
- net MDA46 renamed /MDA46
- net MDA47 renamed /MDA47
- net MDA48 renamed /MDA48
- net MDA49 renamed /MDA49
- net MDA5 renamed /MDA5
- net MDA50 renamed /MDA50
- net MDA51 renamed /MDA51
- net MDA52 renamed /MDA52
- net MDA53 renamed /MDA53
- net MDA54 renamed /MDA54
- net MDA55 renamed /MDA55
- net MDA56 renamed /MDA56
- net MDA57 renamed /MDA57
- net MDA58 renamed /MDA58
- net MDA59 renamed /MDA59
- net MDA6 renamed /MDA6
- net MDA60 renamed /MDA60
- net MDA61 renamed /MDA61
- net MDA62 renamed /MDA62
- net MDA63 renamed /MDA63
- net MDA7 renamed /MDA7
- net MDA8 renamed /MDA8
- net MDA9 renamed /MDA9
- net MDAT renamed /MDAT
- net MDB0 renamed /MDB0
- net MDB1 renamed /MDB1
- net MDB10 renamed /MDB10
- net MDB11 renamed /MDB11
- net MDB12 renamed /MDB12
- net MDB13 renamed /MDB13
- net MDB14 renamed /MDB14
- net MDB15 renamed /MDB15
- net MDB16 renamed /MDB16
- net MDB17 renamed /MDB17
- net MDB18 renamed /MDB18
- net MDB19 renamed /MDB19
- net MDB2 renamed /MDB2
- net MDB20 renamed /MDB20
- net MDB21 renamed /MDB21
- net MDB22 renamed /MDB22
- net MDB23 renamed /MDB23
- net MDB24 renamed /MDB24
- net MDB25 renamed /MDB25
- net MDB26 renamed /MDB26
- net MDB27 renamed /MDB27
- net MDB28 renamed /MDB28
- net MDB29 renamed /MDB29
- net MDB3 renamed /MDB3
- net MDB30 renamed /MDB30
- net MDB31 renamed /MDB31
- net MDB32 renamed /MDB32
- net MDB33 renamed /MDB33
- net MDB34 renamed /MDB34
- net MDB35 renamed /MDB35
- net MDB36 renamed /MDB36
- net MDB37 renamed /MDB37
- net MDB38 renamed /MDB38
- net MDB39 renamed /MDB39
- net MDB4 renamed /MDB4
- net MDB40 renamed /MDB40
- net MDB41 renamed /MDB41
- net MDB42 renamed /MDB42
- net MDB43 renamed /MDB43
- net MDB44 renamed /MDB44
- net MDB45 renamed /MDB45
- net MDB46 renamed /MDB46
- net MDB47 renamed /MDB47
- net MDB48 renamed /MDB48
- net MDB49 renamed /MDB49
- net MDB5 renamed /MDB5
- net MDB50 renamed /MDB50
- net MDB51 renamed /MDB51
- net MDB52 renamed /MDB52
- net MDB53 renamed /MDB53
- net MDB54 renamed /MDB54
- net MDB55 renamed /MDB55
- net MDB56 renamed /MDB56
- net MDB57 renamed /MDB57
- net MDB58 renamed /MDB58
- net MDB59 renamed /MDB59
- net MDB6 renamed /MDB6
- net MDB60 renamed /MDB60
- net MDB61 renamed /MDB61
- net MDB62 renamed /MDB62
- net MDB63 renamed /MDB63
- net MDB7 renamed /MDB7
- net MDB8 renamed /MDB8
- net MDB9 renamed /MDB9
- net MIC1_JD renamed /MIC1_JD
- net MIC1_L renamed /MIC1_L
- net MIC1_R renamed /MIC1_R
- net MIC1_VREFO_L renamed /MIC1_VREFO_L
- net MIC1_VREFO_R renamed /MIC1_VREFO_R
- net MIC2_L renamed /MIC2_L
- net MIC2_R renamed /MIC2_R
- net MIC2_VREFO renamed /MIC2_VREFO
- net MODT_A0 renamed /MODT_A0
- net MODT_A1 renamed /MODT_A1
- net MODT_B0 renamed /MODT_B0
- net MODT_B1 renamed /MODT_B1
- net MPD+ renamed /MPD+
- net MPD- renamed /MPD-
- net MSCLK renamed /MSCLK
- net MSDATA renamed /MSDATA
- net N05264 renamed /N05264
- net N106430987 renamed /N106430987
- net N106430997 renamed /N106430997
- net N106621695 renamed /N106621695
- net N124349601 renamed /N124349601
- net N13760503 renamed /N13760503
- net N144550191 renamed /N144550191
- net N167777391 renamed /N167777391
- net N167780271 renamed /N167780271
- net N168552460 renamed /N168552460
- net N16871456 renamed /N16871456
- net N16871464 renamed /N16871464
- net N16871482 renamed /N16871482
- net N16871486 renamed /N16871486
- net N16871955 renamed /N16871955
- net N16871974 renamed /N16871974
- net N16871979 renamed /N16871979
- net N16871983 renamed /N16871983
- net N16872002 renamed /N16872002
- net N16872076 renamed /N16872076
- net N16872082 renamed /N16872082
- net N16872084 renamed /N16872084
- net N16872096 renamed /N16872096
- net N16872296 renamed /N16872296
- net N16952299 renamed /N16952299
- net N17013037 renamed /N17013037
- net N17076531 renamed /N17076531
- net N17076629 renamed /N17076629
- net N18609742 renamed /N18609742
- net N19130720 renamed /N19130720
- net N21168700 renamed /N21168700
- net N21513130 renamed /N21513130
- net N21513143 renamed /N21513143
- net N22095557 renamed /N22095557
- net N23100246 renamed /N23100246
- net N23891470 renamed /N23891470
- net N23891582 renamed /N23891582
- net N23891733 renamed /N23891733
- net N23891784 renamed /N23891784
- net N23891833 renamed /N23891833
- net N24888999 renamed /N24888999
- net N26626371 renamed /N26626371
- net N28032490 renamed /N28032490
- net N29814820 renamed /N29814820
- net N29818181 renamed /N29818181
- net N30641741 renamed /N30641741
- net N30641932 renamed /N30641932
- net N30641991 renamed /N30641991
- net N30641996 renamed /N30641996
- net N30767566 renamed /N30767566
- net N30880053 renamed /N30880053
- net N31282471 renamed /N31282471
- net N314235640 renamed /N314235640
- net N314238100 renamed /N314238100
- net N31424031117 renamed /N31424031117
- net N32297624 renamed /N32297624
- net N32297700 renamed /N32297700
- net N32555455 renamed /N32555455
- net N32624314 renamed /N32624314
- net N36120215 renamed /N36120215
- net N36283610 renamed /N36283610
- net N36283614 renamed /N36283614
- net N36809121 renamed /N36809121
- net N36809135 renamed /N36809135
- net N37484841 renamed /N37484841
- net N37485205 renamed /N37485205
- net N37485393 renamed /N37485393
- net N38984599 renamed /N38984599
- net N38984604 renamed /N38984604
- net N38984609 renamed /N38984609
- net N38984614 renamed /N38984614
- net N38986900 renamed /N38986900
- net N39004258 renamed /N39004258
- net N39034069 renamed /N39034069
- net N39034071 renamed /N39034071
- net N39036744 renamed /N39036744
- net N39091120 renamed /N39091120
- net N39985561 renamed /N39985561
- net N40003245 renamed /N40003245
- net N40006112 renamed /N40006112
- net N40091692 renamed /N40091692
- net N40744880 renamed /N40744880
- net N40759537 renamed /N40759537
- net N40982210 renamed /N40982210
- net N42038804 renamed /N42038804
- net N42038808 renamed /N42038808
- net N42434761 renamed /N42434761
- net N42434781 renamed /N42434781
- net N43360961 renamed /N43360961
- net N43360989 renamed /N43360989
- net N43544770 renamed /N43544770
- net N43556784 renamed /N43556784
- net N43556809 renamed /N43556809
- net N438310381 renamed /N438310381
- net N438310610 renamed /N438310610
- net N44073325 renamed /N44073325
- net N44080562 renamed /N44080562
- net N44092684 renamed /N44092684
- net N44092686 renamed /N44092686
- net N44092691 renamed /N44092691
- net N44092693 renamed /N44092693
- net N44092761 renamed /N44092761
- net N44937174 renamed /N44937174
- net N44937191 renamed /N44937191
- net N44937210 renamed /N44937210
- net N44937232 renamed /N44937232
- net N44975778 renamed /N44975778
- net N45224102 renamed /N45224102
- net N45319876 renamed /N45319876
- net N47362404 renamed /N47362404
- net N5366609 renamed /N5366609
- net N5366636 renamed /N5366636
- net N53727581 renamed /N53727581
- net N5375288 renamed /N5375288
- net N5375315 renamed /N5375315
- net N55586014 renamed /N55586014
- net N57896148 renamed /N57896148
- net N57985309 renamed /N57985309
- net N57989304 renamed /N57989304
- net N58413975 renamed /N58413975
- net N63447375 renamed /N63447375
- net N68165721 renamed /N68165721
- net N68166469 renamed /N68166469
- net N70643044 renamed /N70643044
- net N775726040 renamed /N775726040
- net N77572638 renamed /N77572638
- net N77572654 renamed /N77572654
- net N79131947 renamed /N79131947
- net N90951725 renamed /N90951725
- net NC_1000 renamed /NC_1000
- net NC_1001 renamed /NC_1001
- net NC_1002 renamed /NC_1002
- net NC_1003 renamed /NC_1003
- net NC_1004 renamed /NC_1004
- net NC_1005 renamed /NC_1005
- net NC_1006 renamed /NC_1006
- net NC_1007 renamed /NC_1007
- net NC_1008 renamed /NC_1008
- net NC_1009 renamed /NC_1009
- net NC_1010 renamed /NC_1010
- net NC_1012 renamed /NC_1012
- net NC_1013 renamed /NC_1013
- net NC_1014 renamed /NC_1014
- net NC_1015 renamed /NC_1015
- net NC_1016 renamed /NC_1016
- net NC_1017 renamed /NC_1017
- net NC_1018 renamed /NC_1018
- net NC_1019 renamed /NC_1019
- net NC_1020 renamed /NC_1020
- net NC_1021 renamed /NC_1021
- net NC_1022 renamed /NC_1022
- net NC_1023 renamed /NC_1023
- net NC_1024 renamed /NC_1024
- net NC_1025 renamed /NC_1025
- net NC_1026 renamed /NC_1026
- net NC_1027 renamed /NC_1027
- net NC_1028 renamed /NC_1028
- net NC_1029 renamed /NC_1029
- net NC_1030 renamed /NC_1030
- net NC_1031 renamed /NC_1031
- net NC_1032 renamed /NC_1032
- net NC_1033 renamed /NC_1033
- net NC_1034 renamed /NC_1034
- net NC_1035 renamed /NC_1035
- net NC_1036 renamed /NC_1036
- net NC_1037 renamed /NC_1037
- net NC_1038 renamed /NC_1038
- net NC_1039 renamed /NC_1039
- net NC_1040 renamed /NC_1040
- net NC_1041 renamed /NC_1041
- net NC_1042 renamed /NC_1042
- net NC_1043 renamed /NC_1043
- net NC_1044 renamed /NC_1044
- net NC_1045 renamed /NC_1045
- net NC_1046 renamed /NC_1046
- net NC_1047 renamed /NC_1047
- net NC_1048 renamed /NC_1048
- net NC_1049 renamed /NC_1049
- net NC_1050 renamed /NC_1050
- net NC_1051 renamed /NC_1051
- net NC_1052 renamed /NC_1052
- net NC_1053 renamed /NC_1053
- net NC_1054 renamed /NC_1054
- net NC_1055 renamed /NC_1055
- net NC_1056 renamed /NC_1056
- net NC_1057 renamed /NC_1057
- net NC_1058 renamed /NC_1058
- net NC_1059 renamed /NC_1059
- net NC_1060 renamed /NC_1060
- net NC_1061 renamed /NC_1061
- net NC_1062 renamed /NC_1062
- net NC_1063 renamed /NC_1063
- net NC_1064 renamed /NC_1064
- net NC_1065 renamed /NC_1065
- net NC_1066 renamed /NC_1066
- net NC_1067 renamed /NC_1067
- net NC_1068 renamed /NC_1068
- net NC_1069 renamed /NC_1069
- net NC_1070 renamed /NC_1070
- net NC_1071 renamed /NC_1071
- net NC_1072 renamed /NC_1072
- net NC_1073 renamed /NC_1073
- net NC_1074 renamed /NC_1074
- net NC_1075 renamed /NC_1075
- net NC_1076 renamed /NC_1076
- net NC_1077 renamed /NC_1077
- net NC_1078 renamed /NC_1078
- net NC_1079 renamed /NC_1079
- net NC_1080 renamed /NC_1080
- net NC_1081 renamed /NC_1081
- net NC_1082 renamed /NC_1082
- net NC_1083 renamed /NC_1083
- net NC_1084 renamed /NC_1084
- net NC_1085 renamed /NC_1085
- net NC_1086 renamed /NC_1086
- net NC_1087 renamed /NC_1087
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Other:
- board outline added: 176.8 x 228 mm

Commit message: .
Parts:
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Connections:
- net /+12V renamed +12V
- net /+12V_LOAD renamed +12V_LOAD
- net /-12V renamed -12V
- net /-CASEOPEN renamed -CASEOPEN
- net /-CSA0 renamed -CSA0
- net /-CSA1 renamed -CSA1
- net /-CSB0 renamed -CSB0
- net /-CSB1 renamed -CSB1
- net /-DCLKA0 renamed -DCLKA0
- net /-DCLKA1 renamed -DCLKA1
- net /-DCLKB0 renamed -DCLKB0
- net /-DCLKB1 renamed -DCLKB1
- net /-DDR3_RST renamed -DDR3_RST
- net /-DQSA0 renamed -DQSA0
- net /-DQSA1 renamed -DQSA1
- net /-DQSA2 renamed -DQSA2
- net /-DQSA3 renamed -DQSA3
- net /-DQSA4 renamed -DQSA4
- net /-DQSA5 renamed -DQSA5
- net /-DQSA6 renamed -DQSA6
- net /-DQSA7 renamed -DQSA7
- net /-DQSB0 renamed -DQSB0
- net /-DQSB1 renamed -DQSB1
- net /-DQSB2 renamed -DQSB2
- net /-DQSB3 renamed -DQSB3
- net /-DQSB4 renamed -DQSB4
- net /-DQSB5 renamed -DQSB5
- net /-DQSB6 renamed -DQSB6
- net /-DQSB7 renamed -DQSB7
- net /-D_GPIO_HRST renamed -D_GPIO_HRST
- net /-HOLD0 renamed -HOLD0
- net /-HOLD1 renamed -HOLD1
- net /-PCIE_RST renamed -PCIE_RST
- net /-PCIRSTIN renamed -PCIRSTIN
- net /-PFMRST2 renamed -PFMRST2
- net /-PROCHOT_CON renamed -PROCHOT_CON
- net /-PSON renamed -PSON
- net /-PVIDALRT renamed -PVIDALRT
- net /-PWRBTSW renamed -PWRBTSW
- net /-PWRBT_1 renamed -PWRBT_1
- net /-RST renamed -RST
- net /-RST_BTN renamed -RST_BTN
- net /-SCASA renamed -SCASA
- net /-SCASB renamed -SCASB
- net /-SPI_CS_1 renamed -SPI_CS_1
- net /-SPI_CS_2 renamed -SPI_CS_2
- net /-SPI_HOLD_B renamed -SPI_HOLD_B
- net /-SPI_HOLD_M renamed -SPI_HOLD_M
- net /-SRASA renamed -SRASA
- net /-SRASB renamed -SRASB
- net /-SWEA renamed -SWEA
- net /-SWEB renamed -SWEB
- net /0_8LEVEL_DDR renamed 0_8LEVEL_DDR
- net /15G renamed 15G
- net /15HG renamed 15HG
- net /1_5LG renamed 1_5LG
- net /28_3VSB renamed 28_3VSB
- net /2_5LEVEL renamed 2_5LEVEL
- net /3VDUAL renamed 3VDUAL
- net /3VDUAL_PCH renamed 3VDUAL_PCH
- net /5VAUX_SW renamed 5VAUX_SW
- net /5VDUAL renamed 5VDUAL
- net /5VSB renamed 5VSB
- net /6609_VCC renamed 6609_VCC
- net /95812_FB renamed 95812_FB
- net /95812_FB_R renamed 95812_FB_R
- net /95812_VDD renamed 95812_VDD
- net /95812_VDDP renamed 95812_VDDP
- net /95812_VIN renamed 95812_VIN
- net /AGND renamed AGND
- net /AJ_A2 renamed AJ_A2
- net /AJ_A5 renamed AJ_A5
- net /AJ_B2 renamed AJ_B2
- net /AJ_B5 renamed AJ_B5
- net /AVDD renamed AVDD
- net /A_-CPURST renamed A_-CPURST
- net /A_-HPRDY renamed A_-HPRDY
- net /A_-PROCHOT renamed A_-PROCHOT
- net /A_-SKTOCC renamed A_-SKTOCC
- net /A_-THRMTRIP renamed A_-THRMTRIP
- net /A_-TRST renamed A_-TRST
- net /A_DDR_COMP0 renamed A_DDR_COMP0
- net /A_DDR_COMP1 renamed A_DDR_COMP1
- net /A_DDR_COMP2 renamed A_DDR_COMP2
- net /A_DMI_0RXN renamed A_DMI_0RXN
- net /A_DMI_0RXP renamed A_DMI_0RXP
- net /A_DMI_0TXN renamed A_DMI_0TXN
- net /A_DMI_0TXP renamed A_DMI_0TXP
- net /A_DMI_1RXN renamed A_DMI_1RXN
- net /A_DMI_1RXP renamed A_DMI_1RXP
- net /A_DMI_1TXN renamed A_DMI_1TXN
- net /A_DMI_1TXP renamed A_DMI_1TXP
- net /A_DMI_2RXN renamed A_DMI_2RXN
- net /A_DMI_2RXP renamed A_DMI_2RXP
- net /A_DMI_2TXN renamed A_DMI_2TXN
- net /A_DMI_2TXP renamed A_DMI_2TXP
- net /A_DMI_3RXN renamed A_DMI_3RXN
- net /A_DMI_3RXP renamed A_DMI_3RXP
- net /A_DMI_3TXN renamed A_DMI_3TXN
- net /A_DMI_3TXP renamed A_DMI_3TXP
- net /A_HSW_CFG_RCOMP renamed A_HSW_CFG_RCOMP
- net /A_PECI renamed A_PECI
- net /A_PMSYNC renamed A_PMSYNC
- net /A_PWR_DEBUG renamed A_PWR_DEBUG
- net /A_SM_VREF renamed A_SM_VREF
- net /A_SO renamed A_SO
- net /A_SYC renamed A_SYC
- net /A_TCK renamed A_TCK
- net /A_TESTLOW_1 renamed A_TESTLOW_1
- net /A_TESTLOW_2 renamed A_TESTLOW_2
- net /BEEP- renamed BEEP-
- net /BOOT renamed BOOT
- net /CEB_N renamed CEB_N
- net /CKEA0 renamed CKEA0
- net /CKEA1 renamed CKEA1
- net /CKEB0 renamed CKEB0
- net /CKEB1 renamed CKEB1
- net /CK_-DOTCLK renamed CK_-DOTCLK
- net /CK_-SRCCLK_PCH renamed CK_-SRCCLK_PCH
- net /CK_-SRCCLK_SATA renamed CK_-SRCCLK_SATA
- net /CK_DOTCLK renamed CK_DOTCLK
- net /CK_SRCCLK_PCH renamed CK_SRCCLK_PCH
- net /CK_SRCCLK_SATA renamed CK_SRCCLK_SATA
- net /COUPON1 renamed COUPON1
- net /COUPON2 renamed COUPON2
- net /CPU_VAXG renamed CPU_VAXG
- net /CPU_VTT_OR renamed CPU_VTT_OR
- net /C_-ACZ_RST renamed C_-ACZ_RST
- net /C_ACZ_BITCLK renamed C_ACZ_BITCLK
- net /C_ACZ_SDIN2 renamed C_ACZ_SDIN2
- net /C_ACZ_SDOUT renamed C_ACZ_SDOUT
- net /C_ACZ_SYNC renamed C_ACZ_SYNC
- net /DCLKA0 renamed DCLKA0
- net /DCLKA1 renamed DCLKA1
- net /DCLKB0 renamed DCLKB0
- net /DCLKB1 renamed DCLKB1
- net /DDRVTT renamed DDRVTT
- net /DDR_15V renamed DDR_15V
- net /DDR_15VIO renamed DDR_15VIO
- net /DDR_EN_CON renamed DDR_EN_CON
- net /DDR_VTT_REF renamed DDR_VTT_REF
- net /DMI_COMP renamed DMI_COMP
- net /DQSA0 renamed DQSA0
- net /DQSA1 renamed DQSA1
- net /DQSA2 renamed DQSA2
- net /DQSA3 renamed DQSA3
- net /DQSA4 renamed DQSA4
- net /DQSA5 renamed DQSA5
- net /DQSA6 renamed DQSA6
- net /DQSA7 renamed DQSA7
- net /DQSB0 renamed DQSB0
- net /DQSB1 renamed DQSB1
- net /DQSB2 renamed DQSB2
- net /DQSB3 renamed DQSB3
- net /DQSB4 renamed DQSB4
- net /DQSB5 renamed DQSB5
- net /DQSB6 renamed DQSB6
- net /DQSB7 renamed DQSB7
- net /FAN1_SET renamed FAN1_SET
- net /FAN1_VOUT renamed FAN1_VOUT
- net /FANIO1 renamed FANIO1
- net /FANIO2 renamed FANIO2
- net /FANPWM1 renamed FANPWM1
- net /FANPWM2 renamed FANPWM2
- net /FAUDIO_JD renamed FAUDIO_JD
- net /FDI_CSYNC renamed FDI_CSYNC
- net /FDI_INT renamed FDI_INT
- net /FDI_RCOMP renamed FDI_RCOMP
- net /FDI_TXN0 renamed FDI_TXN0
- net /FDI_TXN1 renamed FDI_TXN1
- net /FDI_TXP0 renamed FDI_TXP0
- net /FDI_TXP1 renamed FDI_TXP1
- net /FRONT_JD renamed FRONT_JD
- net /FUSEVCC_F renamed FUSEVCC_F
- net /FUSEVCC_R renamed FUSEVCC_R
- net /FUSEVCC_USB3_R3 renamed FUSEVCC_USB3_R3
- net /GND renamed GND
- net /GP24 renamed GP24
- net /GP25 renamed GP25
- net /GP26 renamed GP26
- net /GRCOMP renamed GRCOMP
- net /HD+ renamed HD+
- net /H_SYNC renamed H_SYNC
- net /IO_EN1 renamed IO_EN1
- net /ISEN1 renamed ISEN1
- net /ISEN2 renamed ISEN2
- net /ISEN3 renamed ISEN3
- net /ITE_PWROK1 renamed ITE_PWROK1
- net /IT_AVCC renamed IT_AVCC
- net /IT_VCCH renamed IT_VCCH
- net /JP2 renamed JP2
- net /JP3 renamed JP3
- net /JP4 renamed JP4
- net /JP5 renamed JP5
- net /KBCLK renamed KBCLK
- net /KBDATA renamed KBDATA
- net /KCLK renamed KCLK
- net /KDAT renamed KDAT
- net /L2-L renamed L2-L
- net /L2-R renamed L2-R
- net /L2_L renamed L2_L
- net /L2_R renamed L2_R
- net /LAN_3VDUAL_LED renamed LAN_3VDUAL_LED
- net /LA_-SRCCLK_LAN renamed LA_-SRCCLK_LAN
- net /LA_CLKREQB renamed LA_CLKREQB
- net /LA_DVDD10 renamed LA_DVDD10
- net /LA_LED_ACT_TXRX renamed LA_LED_ACT_TXRX
- net /LA_LED_D2 renamed LA_LED_D2
- net /LA_LED_LINK100 renamed LA_LED_LINK100
- net /LA_LED_LINK1000 renamed LA_LED_LINK1000
- net /LA_MDI0+ renamed LA_MDI0+
- net /LA_MDI0- renamed LA_MDI0-
- net /LA_MDI1+ renamed LA_MDI1+
- net /LA_MDI1- renamed LA_MDI1-
- net /LA_MDI2+ renamed LA_MDI2+
- net /LA_MDI2- renamed LA_MDI2-
- net /LA_MDI3+ renamed LA_MDI3+
- net /LA_MDI3- renamed LA_MDI3-
- net /LA_ML_IN renamed LA_ML_IN
- net /LA_ML_IN_C renamed LA_ML_IN_C
- net /LA_ML_IP renamed LA_ML_IP
- net /LA_ML_IP_C renamed LA_ML_IP_C
- net /LA_ML_ON renamed LA_ML_ON
- net /LA_ML_ON_C renamed LA_ML_ON_C
- net /LA_ML_OP renamed LA_ML_OP
- net /LA_ML_OP_C renamed LA_ML_OP_C
- net /LA_REGOUT renamed LA_REGOUT
- net /LA_RSET renamed LA_RSET
- net /LA_SRCCLK_LAN renamed LA_SRCCLK_LAN
- net /LA_VDD33 renamed LA_VDD33
- net /LA_XTALI renamed LA_XTALI
- net /LA_XTALO renamed LA_XTALO
- net /LG1_1 renamed LG1_1
- net /LG2_1 renamed LG2_1
- net /LG3 renamed LG3
- net /LG3_1 renamed LG3_1
- net /LINE1_JD renamed LINE1_JD
- net /LINE2_L renamed LINE2_L
- net /LINE2_R renamed LINE2_R
- net /LINE2_VREFO renamed LINE2_VREFO
- net /LINE_IN_L renamed LINE_IN_L
- net /LINE_IN_R renamed LINE_IN_R
- net /LINE_O_L renamed LINE_O_L
- net /LINE_O_R renamed LINE_O_R
- net /M2_L renamed M2_L
- net /M2_R renamed M2_R
- net /MAAA0 renamed MAAA0
- net /MAAA1 renamed MAAA1
- net /MAAA10 renamed MAAA10
- net /MAAA11 renamed MAAA11
- net /MAAA12 renamed MAAA12
- net /MAAA13 renamed MAAA13
- net /MAAA14 renamed MAAA14
- net /MAAA15 renamed MAAA15
- net /MAAA2 renamed MAAA2
- net /MAAA3 renamed MAAA3
- net /MAAA4 renamed MAAA4
- net /MAAA5 renamed MAAA5
- net /MAAA6 renamed MAAA6
- net /MAAA7 renamed MAAA7
- net /MAAA8 renamed MAAA8
- net /MAAA9 renamed MAAA9
- net /MAAB0 renamed MAAB0
- net /MAAB1 renamed MAAB1
- net /MAAB10 renamed MAAB10
- net /MAAB11 renamed MAAB11
- net /MAAB12 renamed MAAB12
- net /MAAB13 renamed MAAB13
- net /MAAB14 renamed MAAB14
- net /MAAB15 renamed MAAB15
- net /MAAB2 renamed MAAB2
- net /MAAB3 renamed MAAB3
- net /MAAB4 renamed MAAB4
- net /MAAB5 renamed MAAB5
- net /MAAB6 renamed MAAB6
- net /MAAB7 renamed MAAB7
- net /MAAB8 renamed MAAB8
- net /MAAB9 renamed MAAB9
- net /MB_ID2 renamed MB_ID2
- net /MCLK renamed MCLK
- net /MDA0 renamed MDA0
- net /MDA1 renamed MDA1
- net /MDA10 renamed MDA10
- net /MDA11 renamed MDA11
- net /MDA12 renamed MDA12
- net /MDA13 renamed MDA13
- net /MDA14 renamed MDA14
- net /MDA15 renamed MDA15
- net /MDA16 renamed MDA16
- net /MDA17 renamed MDA17
- net /MDA18 renamed MDA18
- net /MDA19 renamed MDA19
- net /MDA2 renamed MDA2
- net /MDA20 renamed MDA20
- net /MDA21 renamed MDA21
- net /MDA22 renamed MDA22
- net /MDA23 renamed MDA23
- net /MDA24 renamed MDA24
- net /MDA25 renamed MDA25
- net /MDA26 renamed MDA26
- net /MDA27 renamed MDA27
- net /MDA28 renamed MDA28
- net /MDA29 renamed MDA29
- net /MDA3 renamed MDA3
- net /MDA30 renamed MDA30
- net /MDA31 renamed MDA31
- net /MDA32 renamed MDA32
- net /MDA33 renamed MDA33
- net /MDA34 renamed MDA34
- net /MDA35 renamed MDA35
- net /MDA36 renamed MDA36
- net /MDA37 renamed MDA37
- net /MDA38 renamed MDA38
- net /MDA39 renamed MDA39
- net /MDA4 renamed MDA4
- net /MDA40 renamed MDA40
- net /MDA41 renamed MDA41
- net /MDA42 renamed MDA42
- net /MDA43 renamed MDA43
- net /MDA44 renamed MDA44
- net /MDA45 renamed MDA45
- net /MDA46 renamed MDA46
- net /MDA47 renamed MDA47
- net /MDA48 renamed MDA48
- net /MDA49 renamed MDA49
- net /MDA5 renamed MDA5
- net /MDA50 renamed MDA50
- net /MDA51 renamed MDA51
- net /MDA52 renamed MDA52
- net /MDA53 renamed MDA53
- net /MDA54 renamed MDA54
- net /MDA55 renamed MDA55
- net /MDA56 renamed MDA56
- net /MDA57 renamed MDA57
- net /MDA58 renamed MDA58
- net /MDA59 renamed MDA59
- net /MDA6 renamed MDA6
- net /MDA60 renamed MDA60
- net /MDA61 renamed MDA61
- net /MDA62 renamed MDA62
- net /MDA63 renamed MDA63
- net /MDA7 renamed MDA7
- net /MDA8 renamed MDA8
- net /MDA9 renamed MDA9
- net /MDAT renamed MDAT
- net /MDB0 renamed MDB0
- net /MDB1 renamed MDB1
- net /MDB10 renamed MDB10
- net /MDB11 renamed MDB11
- net /MDB12 renamed MDB12
- net /MDB13 renamed MDB13
- net /MDB14 renamed MDB14
- net /MDB15 renamed MDB15
- net /MDB16 renamed MDB16
- net /MDB17 renamed MDB17
- net /MDB18 renamed MDB18
- net /MDB19 renamed MDB19
- net /MDB2 renamed MDB2
- net /MDB20 renamed MDB20
- net /MDB21 renamed MDB21
- net /MDB22 renamed MDB22
- net /MDB23 renamed MDB23
- net /MDB24 renamed MDB24
- net /MDB25 renamed MDB25
- net /MDB26 renamed MDB26
- net /MDB27 renamed MDB27
- net /MDB28 renamed MDB28
- net /MDB29 renamed MDB29
- net /MDB3 renamed MDB3
- net /MDB30 renamed MDB30
- net /MDB31 renamed MDB31
- net /MDB32 renamed MDB32
- net /MDB33 renamed MDB33
- net /MDB34 renamed MDB34
- net /MDB35 renamed MDB35
- net /MDB36 renamed MDB36
- net /MDB37 renamed MDB37
- net /MDB38 renamed MDB38
- net /MDB39 renamed MDB39
- net /MDB4 renamed MDB4
- net /MDB40 renamed MDB40
- net /MDB41 renamed MDB41
- net /MDB42 renamed MDB42
- net /MDB43 renamed MDB43
- net /MDB44 renamed MDB44
- net /MDB45 renamed MDB45
- net /MDB46 renamed MDB46
- net /MDB47 renamed MDB47
- net /MDB48 renamed MDB48
- net /MDB49 renamed MDB49
- net /MDB5 renamed MDB5
- net /MDB50 renamed MDB50
- net /MDB51 renamed MDB51
- net /MDB52 renamed MDB52
- net /MDB53 renamed MDB53
- net /MDB54 renamed MDB54
- net /MDB55 renamed MDB55
- net /MDB56 renamed MDB56
- net /MDB57 renamed MDB57
- net /MDB58 renamed MDB58
- net /MDB59 renamed MDB59
- net /MDB6 renamed MDB6
- net /MDB60 renamed MDB60
- net /MDB61 renamed MDB61
- net /MDB62 renamed MDB62
- net /MDB63 renamed MDB63
- net /MDB7 renamed MDB7
- net /MDB8 renamed MDB8
- net /MDB9 renamed MDB9
- net /MIC1_JD renamed MIC1_JD
- net /MIC1_L renamed MIC1_L
- net /MIC1_R renamed MIC1_R
- net /MIC1_VREFO_L renamed MIC1_VREFO_L
- net /MIC1_VREFO_R renamed MIC1_VREFO_R
- net /MIC2_L renamed MIC2_L
- net /MIC2_R renamed MIC2_R
- net /MIC2_VREFO renamed MIC2_VREFO
- net /MODT_A0 renamed MODT_A0
- net /MODT_A1 renamed MODT_A1
- net /MODT_B0 renamed MODT_B0
- net /MODT_B1 renamed MODT_B1
- net /MPD+ renamed MPD+
- net /MPD- renamed MPD-
- net /MSCLK renamed MSCLK
- net /MSDATA renamed MSDATA
- net /N05264 renamed N05264
- net /N106430987 renamed N106430987
- net /N106430997 renamed N106430997
- net /N106621695 renamed N106621695
- net /N124349601 renamed N124349601
- net /N13760503 renamed N13760503
- net /N144550191 renamed N144550191
- net /N167777391 renamed N167777391
- net /N167780271 renamed N167780271
- net /N168552460 renamed N168552460
- net /N16871456 renamed N16871456
- net /N16871464 renamed N16871464
- net /N16871482 renamed N16871482
- net /N16871486 renamed N16871486
- net /N16871955 renamed N16871955
- net /N16871974 renamed N16871974
- net /N16871979 renamed N16871979
- net /N16871983 renamed N16871983
- net /N16872002 renamed N16872002
- net /N16872076 renamed N16872076
- net /N16872082 renamed N16872082
- net /N16872084 renamed N16872084
- net /N16872096 renamed N16872096
- net /N16872296 renamed N16872296
- net /N16952299 renamed N16952299
- net /N17013037 renamed N17013037
- net /N17076531 renamed N17076531
- net /N17076629 renamed N17076629
- net /N18609742 renamed N18609742
- net /N19130720 renamed N19130720
- net /N21168700 renamed N21168700
- net /N21513130 renamed N21513130
- net /N21513143 renamed N21513143
- net /N22095557 renamed N22095557
- net /N23100246 renamed N23100246
- net /N23891470 renamed N23891470
- net /N23891582 renamed N23891582
- net /N23891733 renamed N23891733
- net /N23891784 renamed N23891784
- net /N23891833 renamed N23891833
- net /N24888999 renamed N24888999
- net /N26626371 renamed N26626371
- net /N28032490 renamed N28032490
- net /N29814820 renamed N29814820
- net /N29818181 renamed N29818181
- net /N30641741 renamed N30641741
- net /N30641932 renamed N30641932
- net /N30641991 renamed N30641991
- net /N30641996 renamed N30641996
- net /N30767566 renamed N30767566
- net /N30880053 renamed N30880053
- net /N31282471 renamed N31282471
- net /N314235640 renamed N314235640
- net /N314238100 renamed N314238100
- net /N31424031117 renamed N31424031117
- net /N32297624 renamed N32297624
- net /N32297700 renamed N32297700
- net /N32555455 renamed N32555455
- net /N32624314 renamed N32624314
- net /N36120215 renamed N36120215
- net /N36283610 renamed N36283610
- net /N36283614 renamed N36283614
- net /N36809121 renamed N36809121
- net /N36809135 renamed N36809135
- net /N37484841 renamed N37484841
- net /N37485205 renamed N37485205
- net /N37485393 renamed N37485393
- net /N38984599 renamed N38984599
- net /N38984604 renamed N38984604
- net /N38984609 renamed N38984609
- net /N38984614 renamed N38984614
- net /N38986900 renamed N38986900
- net /N39004258 renamed N39004258
- net /N39034069 renamed N39034069
- net /N39034071 renamed N39034071
- net /N39036744 renamed N39036744
- net /N39091120 renamed N39091120
- net /N39985561 renamed N39985561
- net /N40003245 renamed N40003245
- net /N40006112 renamed N40006112
- net /N40091692 renamed N40091692
- net /N40744880 renamed N40744880
- net /N40759537 renamed N40759537
- net /N40982210 renamed N40982210
- net /N42038804 renamed N42038804
- net /N42038808 renamed N42038808
- net /N42434761 renamed N42434761
- net /N42434781 renamed N42434781
- net /N43360961 renamed N43360961
- net /N43360989 renamed N43360989
- net /N43544770 renamed N43544770
- net /N43556784 renamed N43556784
- net /N43556809 renamed N43556809
- net /N438310381 renamed N438310381
- net /N438310610 renamed N438310610
- net /N44073325 renamed N44073325
- net /N44080562 renamed N44080562
- net /N44092684 renamed N44092684
- net /N44092686 renamed N44092686
- net /N44092691 renamed N44092691
- net /N44092693 renamed N44092693
- net /N44092761 renamed N44092761
- net /N44937174 renamed N44937174
- net /N44937191 renamed N44937191
- net /N44937210 renamed N44937210
- net /N44937232 renamed N44937232
- net /N44975778 renamed N44975778
- net /N45224102 renamed N45224102
- net /N45319876 renamed N45319876
- net /N47362404 renamed N47362404
- net /N5366609 renamed N5366609
- net /N5366636 renamed N5366636
- net /N53727581 renamed N53727581
- net /N5375288 renamed N5375288
- net /N5375315 renamed N5375315
- net /N55586014 renamed N55586014
- net /N57896148 renamed N57896148
- net /N57985309 renamed N57985309
- net /N57989304 renamed N57989304
- net /N58413975 renamed N58413975
- net /N63447375 renamed N63447375
- net /N68165721 renamed N68165721
- net /N68166469 renamed N68166469
- net /N70643044 renamed N70643044
- net /N775726040 renamed N775726040
- net /N77572638 renamed N77572638
- net /N77572654 renamed N77572654
- net /N79131947 renamed N79131947
- net /N90951725 renamed N90951725
- net /NC_1000 renamed NC_1000
- net /NC_1001 renamed NC_1001
- net /NC_1002 renamed NC_1002
- net /NC_1003 renamed NC_1003
- net /NC_1004 renamed NC_1004
- net /NC_1005 renamed NC_1005
- net /NC_1006 renamed NC_1006
- net /NC_1007 renamed NC_1007
- net /NC_1008 renamed NC_1008
- net /NC_1009 renamed NC_1009
- net /NC_1010 renamed NC_1010
- net /NC_1012 renamed NC_1012
- net /NC_1013 renamed NC_1013
- net /NC_1014 renamed NC_1014
- net /NC_1015 renamed NC_1015
- net /NC_1016 renamed NC_1016
- net /NC_1017 renamed NC_1017
- net /NC_1018 renamed NC_1018
- net /NC_1019 renamed NC_1019
- net /NC_1020 renamed NC_1020
- net /NC_1021 renamed NC_1021
- net /NC_1022 renamed NC_1022
- net /NC_1023 renamed NC_1023
- net /NC_1024 renamed NC_1024
- net /NC_1025 renamed NC_1025
- net /NC_1026 renamed NC_1026
- net /NC_1027 renamed NC_1027
- net /NC_1028 renamed NC_1028
- net /NC_1029 renamed NC_1029
- net /NC_1030 renamed NC_1030
- net /NC_1031 renamed NC_1031
- net /NC_1032 renamed NC_1032
- net /NC_1033 renamed NC_1033
- net /NC_1034 renamed NC_1034
- net /NC_1035 renamed NC_1035
- net /NC_1036 renamed NC_1036
- net /NC_1037 renamed NC_1037
- net /NC_1038 renamed NC_1038
- net /NC_1039 renamed NC_1039
- net /NC_1040 renamed NC_1040
- net /NC_1041 renamed NC_1041
- net /NC_1042 renamed NC_1042
- net /NC_1043 renamed NC_1043
- net /NC_1044 renamed NC_1044
- net /NC_1045 renamed NC_1045
- net /NC_1046 renamed NC_1046
- net /NC_1047 renamed NC_1047
- net /NC_1048 renamed NC_1048
- net /NC_1049 renamed NC_1049
- net /NC_1050 renamed NC_1050
- net /NC_1051 renamed NC_1051
- net /NC_1052 renamed NC_1052
- net /NC_1053 renamed NC_1053
- net /NC_1054 renamed NC_1054
- net /NC_1055 renamed NC_1055
- net /NC_1056 renamed NC_1056
- net /NC_1057 renamed NC_1057
- net /NC_1058 renamed NC_1058
- net /NC_1059 renamed NC_1059
- net /NC_1060 renamed NC_1060
- net /NC_1061 renamed NC_1061
- net /NC_1062 renamed NC_1062
- net /NC_1063 renamed NC_1063
- net /NC_1064 renamed NC_1064
- net /NC_1065 renamed NC_1065
- net /NC_1066 renamed NC_1066
- net /NC_1067 renamed NC_1067
- net /NC_1068 renamed NC_1068
- net /NC_1069 renamed NC_1069
- net /NC_1070 renamed NC_1070
- net /NC_1071 renamed NC_1071
- net /NC_1072 renamed NC_1072
- net /NC_1073 renamed NC_1073
- net /NC_1074 renamed NC_1074
- net /NC_1075 renamed NC_1075
- net /NC_1076 renamed NC_1076
- net /NC_1077 renamed NC_1077
- net /NC_1078 renamed NC_1078
- net /NC_1079 renamed NC_1079
- net /NC_1080 renamed NC_1080
- net /NC_1081 renamed NC_1081
- net /NC_1082 renamed NC_1082
- net /NC_1083 renamed NC_1083
- net /NC_1084 renamed NC_1084
- net /NC_1085 renamed NC_1085
- net /NC_1086 renamed NC_1086
- net /NC_1087 renamed NC_1087
- net /NC_1088 renamed NC_1088
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Other:
- board outline removed
